File: Moteur.sch (KiCad schematic (older format))
At the start: 54 parts, among them IC1 TPS71501, IC2 TLV710, IC3 MAX3051, IC4 LM5106, IC5 LM5106, IC6 INA282, P1 Bus2, P2 MOTOR, P3 GPIO, P4 CONN_1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

Commit message: Start selecting components
Parts:
- removed C1: 100n, ~, symbol C
- removed C11, C12: 10pF, ~, symbol C
- removed C14, C16: 47nF, SM1206, symbol C
- removed C15: 100nF, SM1206, symbol C
- removed C19: 100nF (DNP), ~, symbol C
- removed C2: 100nF, ~, symbol C
- removed C3: 4.7uF, ~, symbol C
- removed C4: 470n, ~, symbol C
- removed D1: DIODESCH, ~, symbol DIODESCH
- removed D3, D4: BAV102, diode-1-SOD80C, symbol DIODE
- removed IC1: TPS71501, symbol TPS71501
- removed IC2: TLV710, symbol TLV710
- removed IC4, IC5: LM5106, symbol LM5106
- removed IC6: INA282, ~, symbol INA282
- removed L1: INDUCTOR, ~, symbol INDUCTOR
- removed P3: GPIO, ~, symbol CONN_7
- removed Q1, Q2, Q3, Q4: IRF8721, transistor-power-SOT669, symbol IRF8721
- removed R1: 5.6M, ~, symbol R
- removed R10: 0.01R, ~, symbol R
- removed R11, R8: 100k, SM0805, symbol R
- removed R2: 910k, ~, symbol R
- removed R3, R5, R6: 10k, ~, symbol R
- removed R9: 330, ~, symbol R
- removed X1: 16MHz, ~, symbol QUARTZCMS4
- added U?: DRV8323RS, symbol cvra:DRV8323RS
- C10, C13, C17, C18, C5, C6, C7, C8, C9: symbol C -> Device:C
- D2: symbol LED -> Device:LED
- IC3: symbol MAX3051 -> Comp2014:MAX3051
- P1: symbol CONN_4 -> phoenix:CONN_4
- P2: symbol CONN_6 -> phoenix:CONN_6
- P4, P6: symbol CONN_1 -> phoenix:CONN_1
- P5: symbol CONN_7 -> phoenix:CONN_7
- R12: value 100k -> 470k; symbol R -> Device:R
- R13: value 18k -> 22k; symbol R -> Device:R
- R4: symbol R -> Device:R
- U1: symbol STM32F303CCT6 -> _stm32:STM32F303CCT6
Connections:
- net labels removed: +5V_PROTECTED, +9V
- wire segments 181 -> 109
- no-connect marks 16 -> 14
Other:
- note added: "6 to 60V Operating Voltage Rang"
- note added: "[Uin (max) = 60V, Uadc max = 3.3V]\nGain K = R13/R12+R13 = 0.9553 (-> 73.8V abs. max)\nFc = 1/K*R12*C18*2pi = 0.76kHz"
- note removed: "3s-4s Lipo\n(9-16.8V)"
- note removed: "8.6V"
- note removed: "Fc = 4.8kHz"
- note removed: "[Uin (max) = 16.8V, Uadc max = 3.3V]\nGain K = R13/R12+R13 = 0.1525 (-> 21.5V abs. max)\nFc = 1/K*R12*C18*2pi = 1kHz"
