File: 3phase.sch (KiCad schematic (older format))
At the start: 21 parts, among them IC3 MAX3051, P1 Bus2, P2 MOTOR, P4 CONN_1, P5 DBG, P6 CONN_1, U1 STM32F303CCT6

Commit message: add FDMD8260L
Parts:
- removed C10: 10n, ~, symbol Device:C
- removed C17, C8: 1uF, ~, symbol Device:C
- removed C5, C6, C7, C9: 100n, ~, symbol Device:C
- removed IC3: MAX3051, ~, symbol Comp2014:MAX3051
- removed U1: STM32F303CCT6, MODULE, symbol _stm32:STM32F303CCT6
- added C? (x2): 0.1uF, ~, symbol Device:C
- added C? (x2): 100nF, ~, symbol Device:C
- added C?: 4.7uF, ~, symbol Device:C
- added C?: 10nF, ~, symbol Device:C
- added C? (x3): 1uF, ~, symbol Device:C
- added C?: 10uF, ~, symbol Device:C
- added Q? (x3): FDMD8260L, symbol cvra:FDMD8260L
- added R? (x3): 5m, symbol Device:R
- added U?: STM32L432KCU, Package_DFN_QFN:QFN-32-1EP_5x5mm_P0.5mm_EP3.45x3.45mm, symbol MCU_ST_STM32L4:STM32L432KCUx
- added U?: LTC2875-DD, Package_DFN_QFN:DFN-8-1EP_3x3mm_P0.5mm_EP1.66x2.38mm, symbol Interface_CAN_LIN:LTC2875-DD
- C13: value 100n -> 0.1uF
Connections:
- net labels added: CAN_RX, CAN_TX, HallA, HallB, HallC, INHA, INHB, INHC, INLA, INLB, INLC, Motor_A, Motor_B, Motor_C, SCLK, SDI, SDO, SOA, SOB, SOC, SWCLK, SWDIO, nSCS
- net labels removed: +3.3V_A, ADC/I_MOT, CAN_SPEED, GPIO_A, GPIO_ADC, GPIO_B, LED, Mot_En_1, Mot_En_2, PWM1, PWM2, Swdclk, Swdio, TESTPT
- wire segments 109 -> 282
- no-connect marks 14 -> 6

Commit message: change MOS drive
Parts:
- removed U?: DRV8323RS, symbol cvra:DRV8323RS
- added U?: DRV8323S, symbol cvra:DRV8323S
Connections:
- wire segments 282 -> 285
- no-connect marks 6 -> 4
Other:
- moved on the sheet: U?

Commit message: first version of the schema completed
Parts:
- removed P1: Bus2, symbol phoenix:CONN_4
- removed P2: MOTOR, ~, symbol phoenix:CONN_6
- removed P5: DBG, symbol phoenix:CONN_7
- added +5V1, GND1, Hall_A1, Hall_B1, Hall_C1, Phase_A1, Phase_B1, Phase_C1: CONN_1, ~, symbol phoenix:CONN_1
- added C6: 1uF, ~, symbol Device:C
- added C7: 10uF, ~, symbol Device:C
- added CONN1: SWD_DEBUG, MODULE, symbol _connectors:SWD_DEBUG
- added CONN2: ENCODER, symbol _connectors:ENCODER
- added CONN3, CONN4: CAN, MODULE, symbol _connectors:CAN
- added U1: MCP1703A-3302_SOT23, Package_TO_SOT_SMD:SOT-23, symbol Regulator_Linear:MCP1703A-3302_SOT23
- gave numbers to parts that had none: 19
- renumbered P6 to Mass1, P4 to Power1
Connections:
- net labels added: Hall_A, Hall_B, Hall_C, Phase_A, Phase_B, Phase_C
- net labels removed: +5V_protected, CANH, CANL, HallA, HallB, HallC, Mot+, Mot-
- wire segments 285 -> 311
Other:
- moved on the sheet: U3

Commit message: schema v0.1
Parts:
- removed +5V1, GND1, Hall_A1, Hall_B1, Hall_C1, Mass1, Phase_A1, Phase_B1, Phase_C1, Power1: CONN_1, ~, symbol phoenix:CONN_1
- added J5: PADS, symbol Connector_Generic:Conn_01x08
- added J6: PADS, symbol Connector_Generic:Conn_01x02
- C1: value 10uF -> >10uF
- C5: value 1uF -> 47nF
- J1: renamed from CONN1; value SWD_DEBUG -> PADS
- J2: renamed from CONN2; value ENCODER -> PICOBLADE
- J3: renamed from CONN3; value CAN -> PICOBLADE
- J4: renamed from CONN4; value CAN -> PICOBLADE
Connections:
- net labels added: ENCODER_A, ENCODER_B, ENCODER_I, HALL_A, HALL_B, HALL_C, PHASE_A, PHASE_B, PHASE_C, RESET, RX, TX
- net labels removed: A, B, Hall_A, Hall_B, Hall_C, I, Motor_A, Motor_B, Motor_C, Phase_A, Phase_B, Phase_C, Reset, Rx, Tx
- wire segments 311 -> 304
Other:
- note added: "6V to 60V Operating Voltage Rang"
- note added: "STM32 internal pull-up"
- note removed: "6 to 60V Operating Voltage Rang"

Commit message: v0.2
Parts:
- removed Q1, Q2: FDMD8260L, symbol cvra:FDMD8260L
- added Q? (x2): FDMD8260L, symbol cvra:FDMD8260L
- R1, R2, R3: value 5m -> ?
Connections:
- wire segments 304 -> 262
Other:
- moved on the sheet: U3

Commit message: multi page + add protection
Parts:
- removed C1: >10uF, ~, symbol Device:C
- removed C10: 4.7uF, ~, symbol Device:C
- removed C11: 10nF, ~, symbol Device:C
- removed C12, C3: 1uF, ~, symbol Device:C
- removed C13, C2, C4: 0.1uF, ~, symbol Device:C
- removed C5: 47nF, ~, symbol Device:C
- removed C8, C9: 100nF, ~, symbol Device:C
- removed J2: PICOBLADE, symbol _connectors:ENCODER
- removed J3, J4: PICOBLADE, MODULE, symbol _connectors:CAN
- removed Q3, Q? (x2): FDMD8260L, symbol cvra:FDMD8260L
- removed R1, R2, R3: ?, symbol Device:R
- removed U2: DRV8323S, symbol cvra:DRV8323S
- removed U3: STM32L432KCU, Package_DFN_QFN:QFN-32-1EP_5x5mm_P0.5mm_EP3.45x3.45mm, symbol MCU_ST_STM32L4:STM32L432KCUx
- removed U4: LTC2875-DD, Package_DFN_QFN:DFN-8-1EP_3x3mm_P0.5mm_EP1.66x2.38mm, symbol Interface_CAN_LIN:LTC2875-DD
- added D1: D_Zener, symbol Device:D_Zener
- added J3, J4: PICOBLADE, MODULE, symbol Connector_Generic:Conn_01x04
- added J5: PADS, symbol Connector_Generic:Conn_01x08
- added Q4, Q?: Q_PMOS_DGS, symbol Device:Q_PMOS_DGS
- added R5: ?, ~, symbol Device:R
- J1: symbol _connectors:SWD_DEBUG -> Connector_Generic:Conn_01x07
- J6: renamed from J5; value PADS -> PICOBLADE; symbol Connector_Generic:Conn_01x08 -> Connector_Generic:Conn_01x05
- renumbered J6 to J2
Connections:
- net labels added: +5V_protected
- net labels removed: ADC/V_BAT, CAN_RX, CAN_TX, ENCODER_A, ENCODER_B, ENCODER_I, HALL_A, HALL_B, HALL_C, INHA, INHB, INHC, INLA, INLB, INLC, PHASE_A, PHASE_B, PHASE_C, RESET, RX, SCLK, SDI, SDO, SOA, SOB, SOC, SWCLK, SWDIO, TX, nSCS
- wire segments 262 -> 79
- no-connect marks 4 -> 0
Other:
- note added: "+3.3V"
- note added: "+5V"
- note added: "+BATT"
- note added: "5V"
- note added: "CANH"
- note added: "CANL"
- note added: "ENCODER_A"
- note added: "ENCODER_B"
- note added: "ENCODER_I"
- note added: "GND"
- note added: "HALL_A"
- note added: "HALL_B"
- note added: "HALL_C"
- note added: "NRST"
- note added: "PHASE_A"
- note added: "PHASE_B"
- note added: "PHASE_C"
- note added: "RX"
- note added: "SWCLK"
- note added: "SWDIO"
- note added: "TX"
- note removed: "STM32 internal pull-up"

Commit message: modif schema
Parts:
- gave numbers to parts that had none: 1
Changed lines of the file:
@@
 	2270 3735 2725 3735
 $Comp
-L Device:Q_PMOS_DGS Q?
+L Device:Q_PMOS_DGS Q5
 U 1 1 5B59B3ED
 P 4155 6830
-F 0 "Q?" V 4498 6830 50  0000 C CNN
+F 0 "Q5" V 4498 6830 50  0000 C CNN
 F 1 "Q_PMOS_DGS" V 4407 6830 50  0000 C CNN
 F 2 "" H 4355 6930 50  0001 C CNN
@@
 	5700 6730 5945 6730
 $Comp
-L power:+5V #PWR?
+L power:+5V #PWR08
 U 1 1 5B5B7BF3
 P 3695 6730
-F 0 "#PWR?" H 3695 6820 20  0001 C CNN
+F 0 "#PWR08" H 3695 6820 20  0001 C CNN
 F 1 "+5V" H 3695 6880 30  0000 C CNN
 F 2 "" H 3695 6730 60  0000 C CNN
@@
 $EndComp
 $Comp
-L power:GND #PWR?
+L power:GND #PWR06
 U 1 1 5B5D1701
 P 2345 7180
-F 0 "#PWR?" H 2345 6930 50  0001 C CNN
+F 0 "#PWR06" H 2345 6930 50  0001 C CNN
 F 1 "GND" H 2345 7030 50  0000 C CNN
 F 2 "" H 2345 7180 50  0001 C CNN
@@
 Connection ~ 5265 7030
 $Comp
-L power:GND #PWR?
+L power:GND #PWR034
 U 1 1 5B603413
 P 5000 7030
-F 0 "#PWR?" H 5000 6780 50  0001 C CNN
+F 0 "#PWR034" H 5000 6780 50  0001 C CNN
 F 1 "GND" H 5000 6880 50  0000 C CNN
 F 2 "" H 5000 7030 50  0001 C CNN
@@
 	5000 7030 5265 7030
 $Comp
-L power:GND #PWR?
+L power:GND #PWR023
 U 1 1 5B60FAAD
 P 4450 1935
-F 0 "#PWR?" H 4450 1685 50  0001 C CNN
+F 0 "#PWR023" H 4450 1685 50  0001 C CNN
 F 1 "GND" H 4450 1785 50  0000 C CNN
 F 2 "" H 4450 1935 50  0001 C CNN
@@
 Connection ~ 4450 1935
 $Comp
-L Comp2014:+5V_protected #PWR?
+L Comp2014:+5V_protected #PWR026
 U 1 1 5B617431
 P 4595 6485
-F 0 "#PWR?" H 4595 6575 20  0001 C CNN
+F 0 "#PWR026" H 4595 6575 20  0001 C CNN
 F 1 "+5V_protected" H 4591 6613 30  0000 C CNN
 F 2 "" H 4595 6485 60  0000 C CNN
@@
 $EndComp
 $Comp
-L Comp2014:+5V_protected #PWR?
+L Comp2014:+5V_protected #PWR038
 U 1 1 5B61F0EB
 P 9385 3935
-F 0 "#PWR?" H 9385 4025 20  0001 C CNN
+F 0 "#PWR038" H 9385 4025 20  0001 C CNN
 F 1 "+5V_protected" V 9382 4033 30  0000 L CNN
 F 2 "" H 9385 3935 60  0000 C CNN
@@
 $EndComp
 $Comp
-L Comp2014:+5V_protected #PWR?
+L Comp2014:+5V_protected #PWR037
 U 1 1 5B62E2CA
 P 9385 3135
-F 0 "#PWR?" H 9385 3225 20  0001 C CNN
+F 0 "#PWR037" H 9385 3225 20  0001 C CNN
 F 1 "+5V_protected" V 9382 3233 30  0000 L CNN
 F 2 "" H 9385 3135 60  0000 C CNN

Commit message: Ĉlean motor-drive schema, add protect and filter
Parts:
- R12: value 470k -> 470kΩ
- R13: value 22k -> 22kΩ
- R4: value 330 -> 330Ω
Other:
- note added: "[Uin (max) = 60V, Uadc max = 3.3V]\nGain K = R13/R12+R13 = 0.0447 (-> 73.8V abs. max)\nFc = 1/K*R12*C18*2pi = 0.76kHz"
- note removed: "[Uin (max) = 60V, Uadc max = 3.3V]\nGain K = R13/R12+R13 = 0.9553 (-> 73.8V abs. max)\nFc = 1/K*R12*C18*2pi = 0.76kHz"
Changed lines of the file:
@@
 P 3290 2485
 F 0 "R4" V 3370 2485 40  0000 C CNN
-F 1 "330" V 3297 2486 40  0000 C CNN
+F 1 "330Ω" V 3297 2486 40  0000 C CNN
 F 2 "~" V 3220 2485 30  0000 C CNN
 F 3 "~" H 3290 2485 30  0000 C CNN
@@
 P 4450 1485
 F 0 "R12" V 4530 1485 40  0000 C CNN
-F 1 "470k" V 4457 1486 40  0000 C CNN
+F 1 "470kΩ" V 4457 1486 40  0000 C CNN
 F 2 "~" V 4380 1485 30  0000 C CNN
 F 3 "~" H 4450 1485 30  0000 C CNN
@@
 P 4450 1785
 F 0 "R13" V 4530 1785 40  0000 C CNN
-F 1 "22k" V 4457 1786 40  0000 C CNN
+F 1 "22kΩ" V 4457 1786 40  0000 C CNN
 F 2 "~" V 4380 1785 30  0000 C CNN
 F 3 "~" H 4450 1785 30  0000 C CNN
@@
 $EndComp
 Text Notes 4560 1135 0    40   ~ 0
-[Uin (max) = 60V, Uadc max = 3.3V]\nGain K = R13/R12+R13 = 0.9553 (-> 73.8V abs. max)\nFc = 1/K*R12*C18*2pi = 0.76kHz
+[Uin (max) = 60V, Uadc max = 3.3V]\nGain K = R13/R12+R13 = 0.0447 (-> 73.8V abs. max)\nFc = 1/K*R12*C18*2pi = 0.76kHz
 $Comp
 L logo:CVRA_logo #G1
