File: 3phase.sch (KiCad schematic (older format))
At the start: 18 parts, among them J1 PADS, J2 PADS, J3 PICOBLADE, J4 PICOBLADE, J5 PADS, J6 PICOBLADE, Q4 Q_PMOS_DGS, Q5 Q_PMOS_DGS, U1 MCP1703A-3302_SOT23

Commit message: clean schema
Parts:
- added FD1, FD2, FD3, FD4: FIDUCIAL_SMD, symbol Mechanical:Mounting_Hole
- added MK1, MK2: Mounting_Hole_PAD, symbol Mechanical:Mounting_Hole_PAD
Changed lines of the file:
@@
 F 3 "" H 2345 6580 60  0000 C CNN
 	1    2345 6580
-	0    1    1    0
+	1    0    0    -1
 $EndComp
 $Comp
@@
 F 3 "" H 5945 6730 60  0000 C CNN
 	1    5945 6730
-	0    1    1    0
+	1    0    0    -1
 $EndComp
 Wire Wire Line
@@
 F 3 "" H 3695 6730 60  0000 C CNN
 	1    3695 6730
-	0    -1   -1   0
+	1    0    0    -1
 $EndComp
 Wire Wire Line
@@
 F 3 "" H 2345 7180 50  0001 C CNN
 	1    2345 7180
-	0    -1   -1   0
+	1    0    0    -1
 $EndComp
 Wire Wire Line
@@
 	0    -1   -1   0
 $EndComp
+$Comp
+L Mechanical:Mounting_Hole_PAD MK1
+U 1 1 5B5B1445
+P 8830 5815
+F 0 "MK1" H 8930 5866 50  0000 L CNN
+F 1 "Mounting_Hole_PAD" H 8930 5775 50  0000 L CNN
+F 2 "" H 8830 5815 50  0001 C CNN
+F 3 "" H 8830 5815 50  0001 C CNN
+	1    8830 5815
+	1    0    0    -1
+$EndComp
+$Comp
+L Mechanical:Mounting_Hole_PAD MK2
+U 1 1 5B5B1526
+P 9885 5815
+F 0 "MK2" H 9985 5866 50  0000 L CNN
+F 1 "Mounting_Hole_PAD" H 9985 5775 50  0000 L CNN
+F 2 "" H 9885 5815 50  0001 C CNN
+F 3 "" H 9885 5815 50  0001 C CNN
+	1    9885 5815
+	1    0    0    -1
+$EndComp
+$Comp
+L power:GND #PWR042
+U 1 1 5B5B3DD0
+P 8830 5915
+F 0 "#PWR042" H 8830 5665 50  0001 C CNN
+F 1 "GND" H 8830 5765 50  0000 C CNN
+F 2 "" H 8830 5915 50  0001 C CNN
+F 3 "" H 8830 5915 50  0001 C CNN
+	1    8830 5915
+	1    0    0    -1
+$EndComp
+$Comp
+L power:GND #PWR043
+U 1 1 5B5B65FC
+P 9885 5915
+F 0 "#PWR043" H 9885 5665 50  0001 C CNN
+F 1 "GND" H 9885 5765 50  0000 C CNN
+F 2 "" H 9885 5915 50  0001 C CNN
+F 3 "" H 9885 5915 50  0001 C CNN
+	1    9885 5915
+	1    0    0    -1
+$EndComp
+$Comp
+L Mechanical:Mounting_Hole FD2
+U 1 1 5B5BB9DE
+P 8865 5110
+F 0 "FD2" H 8965 5156 50  0000 L CNN
+F 1 "FIDUCIAL_SMD" H 8965 5065 50  0000 L CNN
+F 2 "" H 8865 5110 50  0001 C CNN
+F 3 "" H 8865 5110 50  0001 C CNN
+	1    8865 5110
+	1    0    0    -1
+$EndComp
+$Comp
+L Mechanical:Mounting_Hole FD1
+U 1 1 5B5BE32C
+P 8855 5325
+F 0 "FD1" H 8955 5371 50  0000 L CNN
+F 1 "FIDUCIAL_SMD" H 8955 5280 50  0000 L CNN
+F 2 "" H 8855 5325 50  0001 C CNN
+F 3 "" H 8855 5325 50  0001 C CNN
+	1    8855 5325
+	1    0    0    -1
+$EndComp
+$Comp
+L Mechanical:Mounting_Hole FD4
+U 1 1 5B5C341A
+P 9660 5125
+F 0 "FD4" H 9760 5171 50  0000 L CNN
+F 1 "FIDUCIAL_SMD" H 9760 5080 50  0000 L CNN
+F 2 "" H 9660 5125 50  0001 C CNN
+F 3 "" H 9660 5125 50  0001 C CNN
+	1    9660 5125
+	1    0    0    -1
+$EndComp
+$Comp
+L Mechanical:Mounting_Hole FD3
+U 1 1 5B5C3421
+P 9650 5340
+F 0 "FD3" H 9750 5386 50  0000 L CNN
+F 1 "FIDUCIAL_SMD" H 9750 5295 50  0000 L CNN
+F 2 "" H 9650 5340 50  0001 C CNN
+F 3 "" H 9650 5340 50  0001 C CNN
+	1    9650 5340
+	1    0    0    -1
+$EndComp
 $EndSCHEMATC

Commit message: Add solderJumper for encoder
Parts:
- removed J5: PADS, symbol Connector_Generic:Conn_01x08
- added J5: Hole, symbol Connector_Generic:Conn_01x03
- added J7: PICOBLADE, symbol Connector_Generic:Conn_01x05
- added JP1, JP2: SolderJumper_3_Bridged12, symbol Jumper:SolderJumper_3_Bridged12
- J2: value PADS -> Hole
- Q4: value Q_PMOS_DGS -> SQ7415AENW
Connections:
- wire segments 79 -> 81
