File: 3Phase_motor-control.sch (KiCad schematic (older format))
At the start: 8 parts, among them U3 STM32L432KCU, U4 LTC2875-DD

Commit message: clean schema
Changed lines of the file:
@@
 Text HLabel 4175 4295 0    50   Input ~ 0
 SDI
-Text HLabel 4180 4395 0    50   Input ~ 0
+Text HLabel 4175 4395 0    50   Input ~ 0
 TX
-Text HLabel 4180 4495 0    50   Input ~ 0
+Text HLabel 4175 4495 0    50   Input ~ 0
 RX
 Text HLabel 4175 2995 0    50   Input ~ 0
