File: 3Phase_motor-driver.sch (KiCad schematic (older format))
At the start: 12 parts, among them Q1 FDMD8260L, Q2 FDMD8260L, Q3 FDMD8260L, U2 DRV8323S

Commit message: modif schema
Parts:
- removed Q2, Q3: FDMD8260L, symbol cvra:FDMD8260L
- removed R2, R3: ?, symbol Device:R
Connections:
- net labels removed: PHASE_B, PHASE_C
- wire segments 114 -> 65

Commit message: Ĉlean motor-drive schema, add protect and filter
Parts:
- removed R1: ?, symbol Device:R
- added C14, C15, C16: 680pF, ~, symbol Device:C
- added Q2, Q3: FDMD8260L, symbol cvra:FDMD8260L
- added R1, R2, R3: 5mΩ,1W, symbol Device:R_Small
- added R6, R7, R8: 22kΩ, symbol Device:R_Small
- C1: value >10uF -> 15uF,100V
- C2: value 0.1uF -> 0.1uF,X5R,100V
- C4: value 1uF -> 1uF,X5R,16V
- C5: value 47nF -> 47nF,X5R,100V
Connections:
- wire segments 65 -> 89
Other:
- note added: "SOx low-pass filter\nFc = 1 / 2πRC = 10.644 kHz\n"

Commit message: Add solderJumper for encoder
Connections:
- wire segments 89 -> 91
Changed lines of the file:
@@
 Connection ~ 4685 4510
 Connection ~ 4035 4410
+Wire Wire Line
+	6905 1860 7005 1860
+Connection ~ 7005 1860
+Wire Wire Line
+	7105 1860 7005 1860
 $EndSCHEMATC
